File: little-wing.kicad_pcb (KiCad board)
At the start: 2 copper layers, 119.8 x 95.1 mm, 72 parts, among them IC1 AP7335-WG-7, J1 nice!view, J2 Battery, J3 trackball, J4 trackball, SW1 Power, SW2 Reset, U1 nice!nano v2, U2 PMW3610

Commit message: Linking all the main columns together
Routing:
- net Row 2: track 229.9 -> 398.2 mm, vias 16 -> 26
- net Row 1: track 125.1 -> 277.2 mm, vias 7 -> 17
- net Row 0: track 17.5 -> 165.3 mm
- net Col 4: track 123.4 -> 118.2 mm, vias 3 -> 5
- net Col 0: track 209.9 -> 207.9 mm, vias 3 -> 5
- net VCC: track 535.6 -> 534.3 mm
- net Col 2: track 154.2 -> 154.5 mm, vias 3 -> 5
- net Col 3: track 139.1 -> 138.8 mm, vias 3 -> 5
- net Col 1: track 179.2 -> 179.1 mm, vias 3 -> 5
