File: _autosave-little-wing.kicad_pcb (KiCad board)
At the start: 4 copper layers, 207.7 x 119.8 mm, 522 parts, among them IC1 AP7335-WG-7, J1 nice!view, J2 Battery, J3 trackball, J4 rotary, J5 trackball, J6 nice!view, J7 Battery, SW1 Power, SW2 Reset, SW3 Reset, SW4 Power, U1 nice!nano v2, U2 PMW3610, U3 nice!nano v2

Commit message: Making a stack of panels
Parts:
- moved J1 19.3 mm to (190.0, 133.9)
- moved J4 19.3 mm to (201.3, 151.1)
- moved SW1 19.3 mm to (186.9, 141.5)
- moved SW2 19.3 mm to (194.8, 137.7)
- moved U1 19.3 mm to (194.6, 114.0)
- moved J2 19.3 mm to (188.6, 149.9)
Other:
- outline, holes or cut-outs redrawn
Changed lines of the file:
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@@
 	(footprint "Connector_Wuerth:Wuerth_WR-WTB_64800611622_1x06_P1.50mm_Vertical"
 		(layer "F.Cu")
-		(at 220.598 151.634 90)
+		(at 201.294 151.126 90)
 		(descr "Wuerth WR-WTB series connector, 64800611622 (https://katalog.we-online.com/em/datasheet/6480xx11622.pdf), generated with kicad-footprint-generator")
 		(tags "connector Wuerth WR-WTB vertical")
@@
 	(footprint "Connector_PinHeader_2.54mm:PinHeader_1x05_P2.54mm_Vertical"
 		(layer "F.Cu")
-		(at 209.268 134.444 90)
+		(at 189.964 133.936 90)
 		(descr "Through hole straight pin header, 1x05, 2.54mm pitch, single row")
 		(tags "Through hole pin header THT 1x05 2.54mm single row")
@@
 	(footprint "Connector_JST:JST_ZH_S2B-ZR-SM4A-TF_1x02-1MP_P1.50mm_Horizontal"
 		(layer "F.Cu")
-		(at 207.908 150.394 90)
+		(at 188.604 149.886 90)
 		(descr "JST ZH series connector, S2B-ZR-SM4A-TF (http://www.jst-mfg.com/product/pdf/eng/eZH.pdf), generated with kicad-footprint-generator")
 		(tags "connector JST ZH horizontal")
@@
 	(footprint "Button_Switch_SMD:SW_SPDT_PCM12"
 		(layer "F.Cu")
-		(at 206.193 142.034 -90)
+		(at 186.889 141.526 -90)
 		(descr "Ultraminiature Surface Mount Slide Switch, right-angle, https://www.ckswitches.com/media/1424/pcm.pdf")
 		(property "Reference" "SW1"
@@
 	(footprint "Button_Switch_SMD:SW_SPST_B3U-1000P"
 		(layer "F.Cu")
-		(at 214.138 138.244)
+		(at 194.834 137.736)
 		(descr "Ultra-small-sized Tactile Switch with High Contact Reliability, Top-actuated Model, without Ground Terminal, without Boss")
 		(tags "Tactile Switch")
@@
 	(footprint "ScottoKeebs_MCU:Nice_Nano_V2_Flipped"
 		(layer "F.Cu")
-		(at 213.868 114.554)
+		(at 194.564 114.046)
 		(property "Reference" "U1"
 			(at 0 1.625 0)
@@
 	)
 	(gr_arc
-		(start 206.299973 154.308964)
-		(mid 204.87526 153.72885)
-		(end 204.283782 152.308847)
+		(start 186.995973 153.800964)
+		(mid 185.57126 153.22085)
+		(end 184.979782 151.800847)
 		(stroke
 			(width 0.02)
@@
 	)
 	(gr_arc
-		(start 204.284113 98.308944)
-		(mid 204.869907 96.894762)
-		(end 206.284077 96.308967)
+		(start 184.980113 97.800944)
+		(mid 185.565907 96.386762)
+		(end 186.980077 95.800967)
 		(stroke
 			(width 0.02)
@@
 	)
 	(gr_line
-		(start 204.284113 98.308944)
-		(end 204.283782 152.308847)
+		(start 184.980113 97.800944)
+		(end 184.979782 151.800847)
 		(stroke
 			(width 0.02)
@@
 	)
 	(gr_circle
-		(center 213.783771 144.309007)
-		(end 215.033772 144.309007)
+		(center 194.479771 143.801007)
+		(end 195.729772 143.801007)
 		(stroke
 			(width 0.02)
@@
 	)
 	(gr_line
-		(start 221.283648 154.30905)
-		(end 206.299973 154.308964)
+		(start 201.979648 153.80105)
+		(end 186.995973 153.800964)
 		(stroke
 			(width 0.02)
@@
 	)
 	(gr_arc
-		(start 223.283786 152.325214)
-		(mid 222.692231 153.729)
-		(end 221.283648 154.30905)
+		(start 203.979786 151.817214)
+		(mid 203.388231 153.221)
+		(end 201.979648 153.80105)
 		(stroke
 			(width 0.02)
@@
 	)
 	(gr_line
-		(start 206.284077 96.308967)
-		(end 221.284113 96.30905)
+		(start 186.980077 95.800967)
+		(end 201.980113 95.80105)
 		(stroke
 			(width 0.02)
@@
 	)
 	(gr_arc
-		(start 221.284113 96.30905)
-		(mid 222.698408 96.894776)
-		(end 223.284102 98.309064)
+		(start 201.980113 95.80105)
+		(mid 203.394408 96.386776)
+		(end 203.980102 97.801064)
 		(stroke
 			(width 0.02)
@@
 	)
 	(gr_line
-		(start 223.283786 152.325214)
-		(end 223.284102 98.309064)
+		(start 203.979786 151.817214)
+		(end 203.980102 97.801064)
 		(stroke
 			(width 0.02)
