File: kicad/little-wing/sensor.kicad_sch (KiCad schematic)
At the start: 0 parts

Commit message: Re-organising the schematics sheets a bit
Parts:
- added J7: sensor, Connector_JST:JST_SH_SM06B-SRSS-TB_1x06-1MP_P1.00mm_Horizontal, symbol Connector:Conn_01x06_Socket
- added R11, R14, R15, R16: 100R, Resistor_SMD:R_0201_0603Metric, symbol Device:R_Small
Connections:
- new net: J7.2 (Pin_2), R11.2
- new net: J7.5 (Pin_5), R16.2
- new net: J7.3 (Pin_3), R14.2
- new net: J7.4 (Pin_4), R15.2
- new net GND: J7.6 (Pin_6)
- new net Sensor CLK: R15.1
- new net Sensor CS: R11.1
- new net Sensor IRQ: R16.1
- new net Sensor SDIO: R14.1
- new net VDD: J7.1 (Pin_1)
