File: kicad/little-wing/switches.kicad_sch (KiCad schematic)
At the start: 0 parts

Commit message: Re-organising the schematics sheets a bit
Parts:
- added J4: columns, Connector_JST:JST_SH_SM06B-SRSS-TB_1x06-1MP_P1.00mm_Horizontal, symbol Connector:Conn_01x06_Socket
- added J6: rows, Connector_JST:JST_SH_SM05B-SRSS-TB_1x05-1MP_P1.00mm_Horizontal, symbol Connector:Conn_01x05_Socket
Connections:
- new net Col 0: J4.1 (Pin_1)
- new net Col 1: J4.2 (Pin_2)
- new net Col 2: J4.3 (Pin_3)
- new net Col 3: J4.4 (Pin_4)
- new net Col 4: J4.5 (Pin_5)
- new net Col 5: J4.6 (Pin_6)
- new net Row 0: J6.1 (Pin_1)
- new net Row 1: J6.2 (Pin_2)
- new net Row 2: J6.3 (Pin_3)
- new net Row 3: J6.4 (Pin_4)
- new net Row 4: J6.5 (Pin_5)
